File: pcb/schlong_control.sch (KiCad schematic (older format))
At the start: 36 parts, among them P1 Power Connector (120V AC), P2 Input, P3 Output, U1 74HC595, U2 MOC3063M, U3 MOC3063M, U4 MOC3063M, U5 MOC3063M, U6 MOC3063M, U7 LM7805

Commit message: add basic pcb layout
Parts:
- removed U7: LM7805, symbol LM7805
- added 100µF1: Bypass, Capacitors_THT:C_Disc_D3.0mm_W1.6mm_P2.50mm, symbol C
- added U7: LM7805, TO_SOT_Packages_THT:TO-220_Horizontal, symbol 7805_(enumerated_pins)
- C1: footprint (none) -> Capacitors_THT:C_Disc_D3.0mm_W1.6mm_P2.50mm
- D1, D2, D3, D4, D5: footprint (none) -> TO_SOT_Packages_THT:TO-220_Horizontal
- EL-Wire_1, EL-Wire_2, EL-Wire_3, EL-Wire_4, EL-Wire_5, P1: footprint (none) -> Connectors_Terminal_Blocks:TerminalBlock_Pheonix_MKDS1.5-2pol
- P2, P3: footprint (none) -> Connectors:IDC_Header_Straight_10pins
- R1, R10, R11, R12, R13, R14, R15, R2, R3, R4, R5, R6, R7, R8, R9: footprint (none) -> Resistors_THT:R_Axial_DIN0207_L6.3mm_D2.5mm_P7.62mm_Horizontal
- U1: footprint (none) -> Housings_DIP:DIP-16_W7.62mm
- U2, U3, U4, U5, U6: footprint DIP-6 -> Housings_DIP:DIP-6_W7.62mm

Commit message: update pcb
Parts:
- added C2: 0.1uF, symbol C
- C1: value 0.22µF -> 0.33µF
Connections:
- wire segments 132 -> 133
Changed lines of the file:
@@
 Sheet 1 1
 Title "Schlong Module Circuit"
-Date "2017-03-19"
-Rev "3"
+Date "2017-09-01"
+Rev "4"
 Comp "coon@c-base.org"
 Comment1 ""
@@
 AC_P
 $Comp
-L GND #PWR01
+L GND #PWR5
 U 1 1 58A93B28
 P 4850 1550
-F 0 "#PWR01" H 4850 1300 50  0001 C CNN
+F 0 "#PWR5" H 4850 1300 50  0001 C CNN
 F 1 "GND" H 4850 1400 50  0000 C CNN
 F 2 "" H 4850 1550 50  0000 C CNN
@@
 AC_P
 $Comp
-L GND #PWR02
+L GND #PWR6
 U 1 1 58A941CA
 P 4850 2550
-F 0 "#PWR02" H 4850 2300 50  0001 C CNN
+F 0 "#PWR6" H 4850 2300 50  0001 C CNN
 F 1 "GND" H 4850 2400 50  0000 C CNN
 F 2 "" H 4850 2550 50  0000 C CNN
@@
 AC_P
 $Comp
-L GND #PWR03
+L GND #PWR7
 U 1 1 58A94296
 P 4850 3500
-F 0 "#PWR03" H 4850 3250 50  0001 C CNN
+F 0 "#PWR7" H 4850 3250 50  0001 C CNN
 F 1 "GND" H 4850 3350 50  0000 C CNN
 F 2 "" H 4850 3500 50  0000 C CNN
@@
 AC_P
 $Comp
-L GND #PWR04
+L GND #PWR8
 U 1 1 58A94373
 P 4850 4400
-F 0 "#PWR04" H 4850 4150 50  0001 C CNN
+F 0 "#PWR8" H 4850 4150 50  0001 C CNN
 F 1 "GND" H 4850 4250 50  0000 C CNN
 F 2 "" H 4850 4400 50  0000 C CNN
@@
 AC_P
 $Comp
-L GND #PWR05
+L GND #PWR9
 U 1 1 58A94836
 P 4850 5250
-F 0 "#PWR05" H 4850 5000 50  0001 C CNN
+F 0 "#PWR9" H 4850 5000 50  0001 C CNN
 F 1 "GND" H 4850 5100 50  0000 C CNN
 F 2 "" H 4850 5250 50  0000 C CNN
@@
 NoConn ~ 4000 3600
 $Comp
-L VCC #PWR06
+L VCC #PWR3
 U 1 1 58A979A6
 P 1750 2700
-F 0 "#PWR06" H 1750 2550 50  0001 C CNN
+F 0 "#PWR3" H 1750 2550 50  0001 C CNN
 F 1 "VCC" H 1750 2850 50  0000 C CNN
 F 2 "" H 1750 2700 50  0000 C CNN
@@
 $EndComp
 $Comp
-L GND #PWR07
+L GND #PWR4
 U 1 1 58A98202
 P 2450 3700
-F 0 "#PWR07" H 2450 3450 50  0001 C CNN
+F 0 "#PWR4" H 2450 3450 50  0001 C CNN
 F 1 "GND" H 2450 3550 50  0000 C CNN
 F 2 "" H 2450 3700 50  0000 C CNN
@@
 $EndComp
 $Comp
-L PWR_FLAG #FLG08
+L PWR_FLAG #FLG2
 U 1 1 58A91E89
 P 10550 1300
-F 0 "#FLG08" H 10550 1395 50  0001 C CNN
+F 0 "#FLG2" H 10550 1395 50  0001 C CNN
 F 1 "PWR_FLAG" H 10550 1480 50  0000 C CNN
 F 2 "" H 10550 1300 50  0000 C CNN
@@
 $EndComp
 $Comp
-L GND #PWR09
+L GND #PWR20
 U 1 1 58A9369D
 P 10550 1450
-F 0 "#PWR09" H 10550 1200 50  0001 C CNN
+F 0 "#PWR20" H 10550 1200 50  0001 C CNN
 F 1 "GND" H 10550 1300 50  0000 C CNN
 F 2 "" H 10550 1450 50  0000 C CNN
@@
 $EndComp
 $Comp
-L GND #PWR010
+L GND #PWR12
 U 1 1 58C9F740
 P 8100 2900
-F 0 "#PWR010" H 8100 2650 50  0001 C CNN
+F 0 "#PWR12" H 8100 2650 50  0001 C CNN
 F 1 "GND" H 8100 2750 50  0000 C CNN
 F 2 "" H 8100 2900 50  0000 C CNN
@@
 ~LATCH
 $Comp
-L +12V #PWR011
+L +12V #PWR18
 U 1 1 58CA41A9
 P 9750 2200
-F 0 "#PWR011" H 9750 2050 50  0001 C CNN
+F 0 "#PWR18" H 9750 2050 50  0001 C CNN
 F 1 "+12V" H 9750 2340 50  0000 C CNN
 F 2 "" H 9750 2200 50  0000 C CNN
@@
 ~LATCH
 $Comp
-L GND #PWR012
+L GND #PWR19
 U 1 1 58CA466D
 P 9750 2850
-F 0 "#PWR012" H 9750 2600 50  0001 C CNN
+F 0 "#PWR19" H 9750 2600 50  0001 C CNN
 F 1 "GND" H 9750 2700 50  0000 C CNN
 F 2 "" H 9750 2850 50  0000 C CNN
@@
 	9750 2700 9750 2850
 $Comp
-L +12V #PWR013
+L +12V #PWR14
 U 1 1 58CA520E
 P 8800 2100
-F 0 "#PWR013" H 8800 1950 50  0001 C CNN
+F 0 "#PWR14" H 8800 1950 50  0001 C CNN
 F 1 "+12V" H 8800 2240 50  0000 C CNN
 F 2 "" H 8800 2100 50  0000 C CNN
@@
 	8800 2250 8800 2100
 $Comp
-L +12V #PWR014
+L +12V #PWR11
 U 1 1 58C9DC98
 P 8100 2100
-F 0 "#PWR014" H 8100 1950 50  0001 C CNN
+F 0 "#PWR11" H 8100 1950 50  0001 C CNN
 F 1 "+12V" H 8100 2240 50  0000 C CNN
 F 2 "" H 8100 2100 50  0000 C CNN
@@
 ~LATCH
 $Comp
-L GND #PWR015
+L GND #PWR15
 U 1 1 58CA601F
 P 8850 2900
-F 0 "#PWR015" H 8850 2650 50  0001 C CNN
+F 0 "#PWR15" H 8850 2650 50  0001 C CNN
 F 1 "GND" H 8850 2750 50  0000 C CNN
 F 2 "" H 8850 2900 50  0000 C CNN
@@
 	8700 2350 8850 2350
 $Comp
-L +12V #PWR016
+L +12V #PWR21
 U 1 1 58CA7930
 P 10700 2200
-F 0 "#PWR016" H 10700 2050 50  0001 C CNN
+F 0 "#PWR21" H 10700 2050 50  0001 C CNN
 F 1 "+12V" H 10700 2340 50  0000 C CNN
 F 2 "" H 10700 2200 50  0000 C CNN
@@
 	10700 2200 10700 2300
 $Comp
-L GND #PWR017
+L GND #PWR22
 U 1 1 58CA7CF1
 P 10700 2850
-F 0 "#PWR017" H 10700 2600 50  0001 C CNN
+F 0 "#PWR22" H 10700 2600 50  0001 C CNN
 F 1 "GND" H 10700 2700 50  0000 C CNN
 F 2 "" H 10700 2850 50  0000 C CNN
@@
 	9750 2400 9950 2400
 $Comp
-L +12V #PWR018
+L +12V #PWR16
 U 1 1 58CAB532
 P 9000 1250
-F 0 "#PWR018" H 9000 1100 50  0001 C CNN
+F 0 "#PWR16" H 9000 1100 50  0001 C CNN
 F 1 "+12V" H 9000 1390 50  0000 C CNN
 F 2 "" H 9000 1250 50  0000 C CNN
@@
 $EndComp
 $Comp
-L PWR_FLAG #FLG019
+L PWR_FLAG #FLG1
 U 1 1 58CAB634
 P 9350 1300
-F 0 "#FLG019" H 9350 1395 50  0001 C CNN
+F 0 "#FLG1" H 9350 1395 50  0001 C CNN
 F 1 "PWR_FLAG" H 9350 1480 50  0000 C CNN
 F 2 "" H 9350 1300 50  0000 C CNN
@@
 	9350 1400 9350 1300
 $Comp
-L +12V #PWR020
+L +12V #PWR10
 U 1 1 58CAEF1E
 P 7950 3600
-F 0 "#PWR020" H 7950 3450 50  0001 C CNN
+F 0 "#PWR10" H 7950 3450 50  0001 C CNN
 F 1 "+12V" H 7950 3740 50  0000 C CNN
 F 2 "" H 7950 3600 50  0000 C CNN
@@
 	7950 3750 8100 3750
 $Comp
-L GND #PWR021
+L GND #PWR13
 U 1 1 58CAF198
 P 8500 4550
-F 0 "#PWR021" H 8500 4300 50  0001 C CNN
+F 0 "#PWR13" H 8500 4300 50  0001 C CNN
 F 1 "GND" H 8500 4400 50  0000 C CNN
 F 2 "" H 8500 4550 50  0000 C CNN
@@
 	8500 4050 8500 4550
 $Comp
-L VCC #PWR022
+L VCC #PWR17
 U 1 1 58CAF4F3
 P 9150 3600
-F 0 "#PWR022" H 9150 3450 50  0001 C CNN
+F 0 "#PWR17" H 9150 3450 50  0001 C CNN
 F 1 "VCC" H 9150 3750 50  0000 C CNN
 F 2 "" H 9150 3600 50  0000 C CNN
@@
 $EndComp
 Wire Wire Line
-	9150 3750 9150 3600
+	9150 3600 9150 3950
 Wire Wire Line
 	8900 3750 9150 3750
@@
 P 7950 4100
 F 0 "C1" H 7975 4200 50  0000 L CNN
-F 1 "0.22µF" H 7975 4000 50  0000 L CNN
+F 1 "0.33µF" H 7975 4000 50  0000 L CNN
 F 2 "Capacitors_THT:C_Disc_D3.0mm_W1.6mm_P2.50mm" H 7988 3950 50  0001 C CNN
 F 3 "" H 7950 4100 50  0000 C CNN
@@
 	7950 4250 7950 4400
 Wire Wire Line
-	7950 4400 8500 4400
+	7950 4400 9150 4400
 Connection ~ 8500 4400
 $Comp
@@
 $EndComp
 $Comp
-L VCC #PWR023
+L VCC #PWR1
 U 1 1 58CEBA80
 P 1150 3150
-F 0 "#PWR023" H 1150 3000 50  0001 C CNN
+F 0 "#PWR1" H 1150 3000 50  0001 C CNN
 F 1 "VCC" H 1150 3300 50  0000 C CNN
 F 2 "" H 1150 3150 50  0000 C CNN
@@
 $EndComp
 $Comp
-L GND #PWR024
+L GND #PWR2
 U 1 1 58CEBADE
 P 1150 3450
-F 0 "#PWR024" H 1150 3200 50  0001 C CNN
+F 0 "#PWR2" H 1150 3200 50  0001 C CNN
 F 1 "GND" H 1150 3300 50  0000 C CNN
 F 2 "" H 1150 3450 50  0000 C CNN
@@
 	1    0    0    -1
 $EndComp
+$Comp
+L C C2
+U 1 1 59A9C281
+P 9150 4100
+F 0 "C2" H 9175 4200 50  0000 L CNN
+F 1 "0.1uF" H 9175 4000 50  0000 L CNN
+F 2 "" H 9188 3950 50  0001 C CNN
+F 3 "" H 9150 4100 50  0001 C CNN
+	1    9150 4100
+	1    0    0    -1
+$EndComp
+Connection ~ 9150 3750
+Wire Wire Line
+	9150 4400 9150 4250
 $EndSCHEMATC

Commit message: make pcb more compact
Parts:
- C1: footprint Capacitors_THT:C_Disc_D3.0mm_W1.6mm_P2.50mm -> Capacitors_THT:CP_Radial_D4.0mm_P1.50mm
- C2: footprint (none) -> Capacitors_THT:CP_Radial_D4.0mm_P1.50mm
- D1, D2, D3, D4, D5, U7: footprint TO_SOT_Packages_THT:TO-220_Horizontal -> TO_SOT_Packages_THT:TO-220_Vertical
- U2, U3, U4, U5, U6: symbol MOC3063M -> MOC3063M-RESCUE-schlong_control
Changed lines of the file:
@@
 EESchema Schematic File Version 2
+LIBS:schlong_control-rescue
 LIBS:power
 LIBS:device
@@
 LIBS:contrib
 LIBS:valves
-LIBS:bt138
-LIBS:7805_(enumerated_pins)
 LIBS:schlong_control-cache
 EELAYER 25 0
@@
 AC_P
 $Comp
-L GND #PWR5
+L GND #PWR01
 U 1 1 58A93B28
 P 4850 1550
-F 0 "#PWR5" H 4850 1300 50  0001 C CNN
+F 0 "#PWR01" H 4850 1300 50  0001 C CNN
 F 1 "GND" H 4850 1400 50  0000 C CNN
 F 2 "" H 4850 1550 50  0000 C CNN
@@
 AC_P
 $Comp
-L GND #PWR6
+L GND #PWR02
 U 1 1 58A941CA
 P 4850 2550
-F 0 "#PWR6" H 4850 2300 50  0001 C CNN
+F 0 "#PWR02" H 4850 2300 50  0001 C CNN
 F 1 "GND" H 4850 2400 50  0000 C CNN
 F 2 "" H 4850 2550 50  0000 C CNN
@@
 AC_P
 $Comp
-L GND #PWR7
+L GND #PWR03
 U 1 1 58A94296
 P 4850 3500
-F 0 "#PWR7" H 4850 3250 50  0001 C CNN
+F 0 "#PWR03" H 4850 3250 50  0001 C CNN
 F 1 "GND" H 4850 3350 50  0000 C CNN
 F 2 "" H 4850 3500 50  0000 C CNN
@@
 AC_P
 $Comp
-L GND #PWR8
+L GND #PWR04
 U 1 1 58A94373
 P 4850 4400
-F 0 "#PWR8" H 4850 4150 50  0001 C CNN
+F 0 "#PWR04" H 4850 4150 50  0001 C CNN
 F 1 "GND" H 4850 4250 50  0000 C CNN
 F 2 "" H 4850 4400 50  0000 C CNN
@@
 AC_P
 $Comp
-L GND #PWR9
+L GND #PWR05
 U 1 1 58A94836
 P 4850 5250
-F 0 "#PWR9" H 4850 5000 50  0001 C CNN
+F 0 "#PWR05" H 4850 5000 50  0001 C CNN
 F 1 "GND" H 4850 5100 50  0000 C CNN
 F 2 "" H 4850 5250 50  0000 C CNN
@@
 NoConn ~ 4000 3600
 $Comp
-L VCC #PWR3
+L VCC #PWR06
 U 1 1 58A979A6
 P 1750 2700
-F 0 "#PWR3" H 1750 2550 50  0001 C CNN
+F 0 "#PWR06" H 1750 2550 50  0001 C CNN
 F 1 "VCC" H 1750 2850 50  0000 C CNN
 F 2 "" H 1750 2700 50  0000 C CNN
@@
 $EndComp
 $Comp
-L GND #PWR4
+L GND #PWR07
 U 1 1 58A98202
 P 2450 3700
-F 0 "#PWR4" H 2450 3450 50  0001 C CNN
+F 0 "#PWR07" H 2450 3450 50  0001 C CNN
 F 1 "GND" H 2450 3550 50  0000 C CNN
 F 2 "" H 2450 3700 50  0000 C CNN
@@
 $EndComp
 $Comp
-L PWR_FLAG #FLG2
+L PWR_FLAG #FLG08
 U 1 1 58A91E89
 P 10550 1300
-F 0 "#FLG2" H 10550 1395 50  0001 C CNN
+F 0 "#FLG08" H 10550 1395 50  0001 C CNN
 F 1 "PWR_FLAG" H 10550 1480 50  0000 C CNN
 F 2 "" H 10550 1300 50  0000 C CNN
@@
 $EndComp
 $Comp
-L GND #PWR20
+L GND #PWR09
 U 1 1 58A9369D
 P 10550 1450
-F 0 "#PWR20" H 10550 1200 50  0001 C CNN
+F 0 "#PWR09" H 10550 1200 50  0001 C CNN
 F 1 "GND" H 10550 1300 50  0000 C CNN
 F 2 "" H 10550 1450 50  0000 C CNN
@@
 AC_N
 $Comp
-L MOC3063M U2
+L MOC3063M-RESCUE-schlong_control U2
 U 1 1 58B4C29D
 P 5350 1250
@@
 $EndComp
 $Comp
-L MOC3063M U3
+L MOC3063M-RESCUE-schlong_control U3
 U 1 1 58B4C496
 P 5350 2250
@@
 $EndComp
 $Comp
-L MOC3063M U4
+L MOC3063M-RESCUE-schlong_control U4
 U 1 1 58B4C537
 P 5350 3200
@@
 $EndComp
 $Comp
-L MOC3063M U5
+L MOC3063M-RESCUE-schlong_control U5
 U 1 1 58B4C59C
 P 5350 4100
@@
 $EndComp
 $Comp
-L MOC3063M U6
+L MOC3063M-RESCUE-schlong_control U6
 U 1 1 58B4C5FD
 P 5350 4950
@@
 $EndComp
 $Comp
-L GND #PWR12
+L GND #PWR010
 U 1 1 58C9F740
 P 8100 2900
-F 0 "#PWR12" H 8100 2650 50  0001 C CNN
+F 0 "#PWR010" H 8100 2650 50  0001 C CNN
 F 1 "GND" H 8100 2750 50  0000 C CNN
 F 2 "" H 8100 2900 50  0000 C CNN
@@
 ~LATCH
 $Comp
-L +12V #PWR18
+L +12V #PWR011
 U 1 1 58CA41A9
 P 9750 2200
-F 0 "#PWR18" H 9750 2050 50  0001 C CNN
+F 0 "#PWR011" H 9750 2050 50  0001 C CNN
 F 1 "+12V" H 9750 2340 50  0000 C CNN
 F 2 "" H 9750 2200 50  0000 C CNN
@@
 ~LATCH
 $Comp
-L GND #PWR19
+L GND #PWR012
 U 1 1 58CA466D
 P 9750 2850
-F 0 "#PWR19" H 9750 2600 50  0001 C CNN
+F 0 "#PWR012" H 9750 2600 50  0001 C CNN
 F 1 "GND" H 9750 2700 50  0000 C CNN
 F 2 "" H 9750 2850 50  0000 C CNN
@@
 	9750 2700 9750 2850
 $Comp
-L +12V #PWR14
+L +12V #PWR013
 U 1 1 58CA520E
 P 8800 2100
-F 0 "#PWR14" H 8800 1950 50  0001 C CNN
+F 0 "#PWR013" H 8800 1950 50  0001 C CNN
 F 1 "+12V" H 8800 2240 50  0000 C CNN
 F 2 "" H 8800 2100 50  0000 C CNN
@@
 	8800 2250 8800 2100
 $Comp
-L +12V #PWR11
+L +12V #PWR014
 U 1 1 58C9DC98
 P 8100 2100
-F 0 "#PWR11" H 8100 1950 50  0001 C CNN
+F 0 "#PWR014" H 8100 1950 50  0001 C CNN
 F 1 "+12V" H 8100 2240 50  0000 C CNN
 F 2 "" H 8100 2100 50  0000 C CNN
@@
 ~LATCH
 $Comp
-L GND #PWR15
+L GND #PWR015
 U 1 1 58CA601F
 P 8850 2900
-F 0 "#PWR15" H 8850 2650 50  0001 C CNN
+F 0 "#PWR015" H 8850 2650 50  0001 C CNN
 F 1 "GND" H 8850 2750 50  0000 C CNN
 F 2 "" H 8850 2900 50  0000 C CNN
@@
 	8700 2350 8850 2350
 $Comp
-L +12V #PWR21
+L +12V #PWR016
 U 1 1 58CA7930
 P 10700 2200
-F 0 "#PWR21" H 10700 2050 50  0001 C CNN
+F 0 "#PWR016" H 10700 2050 50  0001 C CNN
 F 1 "+12V" H 10700 2340 50  0000 C CNN
 F 2 "" H 10700 2200 50  0000 C CNN
@@
 	10700 2200 10700 2300
 $Comp
-L GND #PWR22
+L GND #PWR017
 U 1 1 58CA7CF1
 P 10700 2850
-F 0 "#PWR22" H 10700 2600 50  0001 C CNN
+F 0 "#PWR017" H 10700 2600 50  0001 C CNN
 F 1 "GND" H 10700 2700 50  0000 C CNN
 F 2 "" H 10700 2850 50  0000 C CNN
@@
 	9750 2400 9950 2400
 $Comp
-L +12V #PWR16
+L +12V #PWR018
 U 1 1 58CAB532
 P 9000 1250
-F 0 "#PWR16" H 9000 1100 50  0001 C CNN
+F 0 "#PWR018" H 9000 1100 50  0001 C CNN
 F 1 "+12V" H 9000 1390 50  0000 C CNN
 F 2 "" H 9000 1250 50  0000 C CNN
@@
 $EndComp
 $Comp
-L PWR_FLAG #FLG1
+L PWR_FLAG #FLG019
 U 1 1 58CAB634
 P 9350 1300
-F 0 "#FLG1" H 9350 1395 50  0001 C CNN
+F 0 "#FLG019" H 9350 1395 50  0001 C CNN
 F 1 "PWR_FLAG" H 9350 1480 50  0000 C CNN
 F 2 "" H 9350 1300 50  0000 C CNN
@@
 	9350 1400 9350 1300
 $Comp
-L +12V #PWR10
+L +12V #PWR020
 U 1 1 58CAEF1E
 P 7950 3600
-F 0 "#PWR10" H 7950 3450 50  0001 C CNN
+F 0 "#PWR020" H 7950 3450 50  0001 C CNN
 F 1 "+12V" H 7950 3740 50  0000 C CNN
 F 2 "" H 7950 3600 50  0000 C CNN
@@
 	7950 3750 8100 3750
 $Comp
-L GND #PWR13
+L GND #PWR021
 U 1 1 58CAF198
 P 8500 4550
-F 0 "#PWR13" H 8500 4300 50  0001 C CNN
+F 0 "#PWR021" H 8500 4300 50  0001 C CNN
 F 1 "GND" H 8500 4400 50  0000 C CNN
 F 2 "" H 8500 4550 50  0000 C CNN
@@
 	8500 4050 8500 4550
 $Comp
-L VCC #PWR17
+L VCC #PWR022
 U 1 1 58CAF4F3
 P 9150 3600
-F 0 "#PWR17" H 9150 3450 50  0001 C CNN
+F 0 "#PWR022" H 9150 3450 50  0001 C CNN
 F 1 "VCC" H 9150 3750 50  0000 C CNN
 F 2 "" H 9150 3600 50  0000 C CNN
@@
 F 0 "C1" H 7975 4200 50  0000 L CNN
 F 1 "0.33µF" H 7975 4000 50  0000 L CNN
-F 2 "Capacitors_THT:C_Disc_D3.0mm_W1.6mm_P2.50mm" H 7988 3950 50  0001 C CNN
+F 2 "Capacitors_THT:CP_Radial_D4.0mm_P1.50mm" H 7988 3950 50  0001 C CNN
 F 3 "" H 7950 4100 50  0000 C CNN
 	1    7950 4100
@@
 F 0 "D1" H 6525 1275 50  0000 L CNN
 F 1 "BT138" H 6525 1200 50  0000 L CNN
-F 2 "TO_SOT_Packages_THT:TO-220_Horizontal" V 6475 1275 50  0001 C CNN
+F 2 "TO_SOT_Packages_THT:TO-220_Vertical" V 6475 1275 50  0001 C CNN
 F 3 "" V 6400 1250 50  0000 C CNN
 	1    6400 1250
@@
 F 0 "D2" H 6525 2275 50  0000 L CNN
 F 1 "BT138" H 6525 2200 50  0000 L CNN
-F 2 "TO_SOT_Packages_THT:TO-220_Horizontal" V 6475 2275 50  0001 C CNN
+F 2 "TO_SOT_Packages_THT:TO-220_Vertical" V 6475 2275 50  0001 C CNN
 F 3 "" V 6400 2250 50  0000 C CNN
 	1    6400 2250
@@
 F 0 "D3" H 6525 3225 50  0000 L CNN
 F 1 "BT138" H 6525 3150 50  0000 L CNN
-F 2 "TO_SOT_Packages_THT:TO-220_Horizontal" V 6475 3225 50  0001 C CNN
+F 2 "TO_SOT_Packages_THT:TO-220_Vertical" V 6475 3225 50  0001 C CNN
 F 3 "" V 6400 3200 50  0000 C CNN
 	1    6400 3200
@@
 F 0 "D4" H 6525 4125 50  0000 L CNN
 F 1 "BT138" H 6525 4050 50  0000 L CNN
-F 2 "TO_SOT_Packages_THT:TO-220_Horizontal" V 6475 4125 50  0001 C CNN
+F 2 "TO_SOT_Packages_THT:TO-220_Vertical" V 6475 4125 50  0001 C CNN
 F 3 "" V 6400 4100 50  0000 C CNN
 	1    6400 4100
@@
 F 0 "D5" H 6525 4975 50  0000 L CNN
 F 1 "BT138" H 6525 4900 50  0000 L CNN
-F 2 "TO_SOT_Packages_THT:TO-220_Horizontal" V 6475 4975 50  0001 C CNN
+F 2 "TO_SOT_Packages_THT:TO-220_Vertical" V 6475 4975 50  0001 C CNN
 F 3 "" V 6400 4950 50  0000 C CNN
 	1    6400 4950
@@
 $EndComp
 $Comp
-L VCC #PWR1
+L VCC #PWR023
 U 1 1 58CEBA80
 P 1150 3150
-F 0 "#PWR1" H 1150 3000 50  0001 C CNN
+F 0 "#PWR023" H 1150 3000 50  0001 C CNN
 F 1 "VCC" H 1150 3300 50  0000 C CNN
 F 2 "" H 1150 3150 50  0000 C CNN
@@
 $EndComp
 $Comp
-L GND #PWR2
+L GND #PWR024
 U 1 1 58CEBADE
 P 1150 3450
-F 0 "#PWR2" H 1150 3200 50  0001 C CNN
+F 0 "#PWR024" H 1150 3200 50  0001 C CNN
 F 1 "GND" H 1150 3300 50  0000 C CNN
 F 2 "" H 1150 3450 50  0000 C CNN
@@
 F 0 "U7" H 8650 3604 50  0000 C CNN
 F 1 "LM7805" H 8500 4000 50  0000 C CNN
-F 2 "TO_SOT_Packages_THT:TO-220_Horizontal" H 8500 3800 50  0001 C CNN
+F 2 "TO_SOT_Packages_THT:TO-220_Vertical" H 8500 3800 50  0001 C CNN
 F 3 "" H 8500 3800 50  0000 C CNN
 	1    8500 3800
@@
 F 0 "C2" H 9175 4200 50  0000 L CNN
 F 1 "0.1uF" H 9175 4000 50  0000 L CNN
-F 2 "" H 9188 3950 50  0001 C CNN
+F 2 "Capacitors_THT:CP_Radial_D4.0mm_P1.50mm" H 9188 3950 50  0001 C CNN
 F 3 "" H 9150 4100 50  0001 C CNN
 	1    9150 4100
